Commit message: Added 4 robots simulation and initial documentation

File: ke_ws/src/panda_multiple_arms/robot_description/panda_multiple_arms.urdf (robot description, URDF)
Before this commit: robot panda_multiple_arms, 46 links, 45 joints
Links:
- removed link left_arm_hand
- removed link left_arm_hand_sc
- removed link left_arm_hand_tcp
- removed link left_arm_leftfinger
- removed link left_arm_link0
- removed link left_arm_link0_sc
- removed link left_arm_link1
- removed link left_arm_link1_sc
- removed link left_arm_link2
- removed link left_arm_link2_sc
- removed link left_arm_link3
- removed link left_arm_link3_sc
- removed link left_arm_link4
- removed link left_arm_link4_sc
- removed link left_arm_link5
- removed link left_arm_link5_sc
- removed link left_arm_link6
- removed link left_arm_link6_sc
- removed link left_arm_link7
- removed link left_arm_link7_sc
- removed link left_arm_link8
- removed link left_arm_rightfinger
- removed link right_arm_hand
- removed link right_arm_hand_sc
- removed link right_arm_hand_tcp
- removed link right_arm_leftfinger
- removed link right_arm_link0
- removed link right_arm_link0_sc
- removed link right_arm_link1
- removed link right_arm_link1_sc
- removed link right_arm_link2
- removed link right_arm_link2_sc
- removed link right_arm_link3
- removed link right_arm_link3_sc
- removed link right_arm_link4
- removed link right_arm_link4_sc
- removed link right_arm_link5
- removed link right_arm_link5_sc
- removed link right_arm_link6
- removed link right_arm_link6_sc
- removed link right_arm_link7
- removed link right_arm_link7_sc
- removed link right_arm_link8
- removed link right_arm_rightfinger
- added link front_left_arm_hand, mass 0.73; collision mesh filename=package://franka_description/meshes/collision/hand.stl; visual mesh filename=package://franka_description/meshes/visual/hand.dae
- added link front_left_arm_hand_sc
- added link front_left_arm_hand_tcp
- added link front_left_arm_leftfinger, mass 0.015; collision box size=17.5e-3 15.2e-3 18.5e-3; collision box size=17.5e-3 7e-3 23.5e-3
- added link front_left_arm_link0, mass 0.629769; collision mesh filename=package://franka_description/meshes/collision/link0.stl; visual mesh filename=package://franka_description/meshes/visual/link0.dae
- added link front_left_arm_link0_sc
- added link front_left_arm_link1, mass 4.970684; collision mesh filename=package://franka_description/meshes/collision/link1.stl; visual mesh filename=package://franka_description/meshes/visual/link1.dae
- added link front_left_arm_link1_sc
- added link front_left_arm_link2, mass 0.646926; collision mesh filename=package://franka_description/meshes/collision/link2.stl; visual mesh filename=package://franka_description/meshes/visual/link2.dae
- added link front_left_arm_link2_sc
- added link front_left_arm_link3, mass 3.228604; collision mesh filename=package://franka_description/meshes/collision/link3.stl; visual mesh filename=package://franka_description/meshes/visual/link3.dae
- added link front_left_arm_link3_sc
- added link front_left_arm_link4, mass 3.587895; collision mesh filename=package://franka_description/meshes/collision/link4.stl; visual mesh filename=package://franka_description/meshes/visual/link4.dae
- added link front_left_arm_link4_sc
- added link front_left_arm_link5, mass 1.225946; collision mesh filename=package://franka_description/meshes/collision/link5.stl; visual mesh filename=package://franka_description/meshes/visual/link5.dae
- added link front_left_arm_link5_sc
- added link front_left_arm_link6, mass 1.666555; collision mesh filename=package://franka_description/meshes/collision/link6.stl; visual mesh filename=package://franka_description/meshes/visual/link6.dae
- added link front_left_arm_link6_sc
- added link front_left_arm_link7, mass 0.735522; collision mesh filename=package://franka_description/meshes/collision/link7.stl; visual mesh filename=package://franka_description/meshes/visual/link7.dae
- added link front_left_arm_link7_sc
- added link front_left_arm_link8
- added link front_left_arm_rightfinger, mass 0.015; collision box size=17.5e-3 15.2e-3 18.5e-3; collision box size=17.5e-3 7e-3 23.5e-3
- added link front_right_arm_hand, mass 0.73; collision mesh filename=package://franka_description/meshes/collision/hand.stl; visual mesh filename=package://franka_description/meshes/visual/hand.dae
- added link front_right_arm_hand_sc
- added link front_right_arm_hand_tcp
- added link front_right_arm_leftfinger, mass 0.015; collision box size=17.5e-3 15.2e-3 18.5e-3; collision box size=17.5e-3 7e-3 23.5e-3
- added link front_right_arm_link0, mass 0.629769; collision mesh filename=package://franka_description/meshes/collision/link0.stl; visual mesh filename=package://franka_description/meshes/visual/link0.dae
- added link front_right_arm_link0_sc
- added link front_right_arm_link1, mass 4.970684; collision mesh filename=package://franka_description/meshes/collision/link1.stl; visual mesh filename=package://franka_description/meshes/visual/link1.dae
- added link front_right_arm_link1_sc
- added link front_right_arm_link2, mass 0.646926; collision mesh filename=package://franka_description/meshes/collision/link2.stl; visual mesh filename=package://franka_description/meshes/visual/link2.dae
- added link front_right_arm_link2_sc
- added link front_right_arm_link3, mass 3.228604; collision mesh filename=package://franka_description/meshes/collision/link3.stl; visual mesh filename=package://franka_description/meshes/visual/link3.dae
- added link front_right_arm_link3_sc
- added link front_right_arm_link4, mass 3.587895; collision mesh filename=package://franka_description/meshes/collision/link4.stl; visual mesh filename=package://franka_description/meshes/visual/link4.dae
- added link front_right_arm_link4_sc
- added link front_right_arm_link5, mass 1.225946; collision mesh filename=package://franka_description/meshes/collision/link5.stl; visual mesh filename=package://franka_description/meshes/visual/link5.dae
- added link front_right_arm_link5_sc
- added link front_right_arm_link6, mass 1.666555; collision mesh filename=package://franka_description/meshes/collision/link6.stl; visual mesh filename=package://franka_description/meshes/visual/link6.dae
- added link front_right_arm_link6_sc
- added link front_right_arm_link7, mass 0.735522; collision mesh filename=package://franka_description/meshes/collision/link7.stl; visual mesh filename=package://franka_description/meshes/visual/link7.dae
- added link front_right_arm_link7_sc
- added link front_right_arm_link8
- added link front_right_arm_rightfinger, mass 0.015; collision box size=17.5e-3 15.2e-3 18.5e-3; collision box size=17.5e-3 7e-3 23.5e-3
- added link rear_left_arm_hand, mass 0.73; collision mesh filename=package://franka_description/meshes/collision/hand.stl; visual mesh filename=package://franka_description/meshes/visual/hand.dae
- added link rear_left_arm_hand_sc
- added link rear_left_arm_hand_tcp
- added link rear_left_arm_leftfinger, mass 0.015; collision box size=17.5e-3 15.2e-3 18.5e-3; collision box size=17.5e-3 7e-3 23.5e-3
- added link rear_left_arm_link0, mass 0.629769; collision mesh filename=package://franka_description/meshes/collision/link0.stl; visual mesh filename=package://franka_description/meshes/visual/link0.dae
- added link rear_left_arm_link0_sc
- added link rear_left_arm_link1, mass 4.970684; collision mesh filename=package://franka_description/meshes/collision/link1.stl; visual mesh filename=package://franka_description/meshes/visual/link1.dae
- added link rear_left_arm_link1_sc
- added link rear_left_arm_link2, mass 0.646926; collision mesh filename=package://franka_description/meshes/collision/link2.stl; visual mesh filename=package://franka_description/meshes/visual/link2.dae
- added link rear_left_arm_link2_sc
- added link rear_left_arm_link3, mass 3.228604; collision mesh filename=package://franka_description/meshes/collision/link3.stl; visual mesh filename=package://franka_description/meshes/visual/link3.dae
- added link rear_left_arm_link3_sc
- added link rear_left_arm_link4, mass 3.587895; collision mesh filename=package://franka_description/meshes/collision/link4.stl; visual mesh filename=package://franka_description/meshes/visual/link4.dae
- added link rear_left_arm_link4_sc
- added link rear_left_arm_link5, mass 1.225946; collision mesh filename=package://franka_description/meshes/collision/link5.stl; visual mesh filename=package://franka_description/meshes/visual/link5.dae
- added link rear_left_arm_link5_sc
- added link rear_left_arm_link6, mass 1.666555; collision mesh filename=package://franka_description/meshes/collision/link6.stl; visual mesh filename=package://franka_description/meshes/visual/link6.dae
- added link rear_left_arm_link6_sc
- added link rear_left_arm_link7, mass 0.735522; collision mesh filename=package://franka_description/meshes/collision/link7.stl; visual mesh filename=package://franka_description/meshes/visual/link7.dae
- added link rear_left_arm_link7_sc
- added link rear_left_arm_link8
- added link rear_left_arm_rightfinger, mass 0.015; collision box size=17.5e-3 15.2e-3 18.5e-3; collision box size=17.5e-3 7e-3 23.5e-3
- added link rear_right_arm_hand, mass 0.73; collision mesh filename=package://franka_description/meshes/collision/hand.stl; visual mesh filename=package://franka_description/meshes/visual/hand.dae
- added link rear_right_arm_hand_sc
- added link rear_right_arm_hand_tcp
- added link rear_right_arm_leftfinger, mass 0.015; collision box size=17.5e-3 15.2e-3 18.5e-3; collision box size=17.5e-3 7e-3 23.5e-3
- added link rear_right_arm_link0, mass 0.629769; collision mesh filename=package://franka_description/meshes/collision/link0.stl; visual mesh filename=package://franka_description/meshes/visual/link0.dae
- added link rear_right_arm_link0_sc
- added link rear_right_arm_link1, mass 4.970684; collision mesh filename=package://franka_description/meshes/collision/link1.stl; visual mesh filename=package://franka_description/meshes/visual/link1.dae
- added link rear_right_arm_link1_sc
- added link rear_right_arm_link2, mass 0.646926; collision mesh filename=package://franka_description/meshes/collision/link2.stl; visual mesh filename=package://franka_description/meshes/visual/link2.dae
- added link rear_right_arm_link2_sc
- added link rear_right_arm_link3, mass 3.228604; collision mesh filename=package://franka_description/meshes/collision/link3.stl; visual mesh filename=package://franka_description/meshes/visual/link3.dae
- added link rear_right_arm_link3_sc
- added link rear_right_arm_link4, mass 3.587895; collision mesh filename=package://franka_description/meshes/collision/link4.stl; visual mesh filename=package://franka_description/meshes/visual/link4.dae
- added link rear_right_arm_link4_sc
- added link rear_right_arm_link5, mass 1.225946; collision mesh filename=package://franka_description/meshes/collision/link5.stl; visual mesh filename=package://franka_description/meshes/visual/link5.dae
- added link rear_right_arm_link5_sc
- added link rear_right_arm_link6, mass 1.666555; collision mesh filename=package://franka_description/meshes/collision/link6.stl; visual mesh filename=package://franka_description/meshes/visual/link6.dae
- added link rear_right_arm_link6_sc
- added link rear_right_arm_link7, mass 0.735522; collision mesh filename=package://franka_description/meshes/collision/link7.stl; visual mesh filename=package://franka_description/meshes/visual/link7.dae
- added link rear_right_arm_link7_sc
- added link rear_right_arm_link8
- added link rear_right_arm_rightfinger, mass 0.015; collision box size=17.5e-3 15.2e-3 18.5e-3; collision box size=17.5e-3 7e-3 23.5e-3
- link base: mass 10.0 -> 20.0; geometry collision box size=2 2 1; visual box size=2 2 1
Joints:
- removed joint left_arm_finger_joint1
- removed joint left_arm_finger_joint2
- removed joint left_arm_hand_joint
- removed joint left_arm_hand_sc_joint
- removed joint left_arm_hand_tcp_joint
- removed joint left_arm_joint1
- removed joint left_arm_joint2
- removed joint left_arm_joint3
- removed joint left_arm_joint4
- removed joint left_arm_joint5
- removed joint left_arm_joint6
- removed joint left_arm_joint7
- removed joint left_arm_joint8
- removed joint left_arm_joint_base
- removed joint left_arm_link0_sc_joint
- removed joint left_arm_link1_sc_joint
- removed joint left_arm_link2_sc_joint
- removed joint left_arm_link3_sc_joint
- removed joint left_arm_link4_sc_joint
- removed joint left_arm_link5_sc_joint
- removed joint left_arm_link6_sc_joint
- removed joint left_arm_link7_sc_joint
- removed joint right_arm_finger_joint1
- removed joint right_arm_finger_joint2
- removed joint right_arm_hand_joint
- removed joint right_arm_hand_sc_joint
- removed joint right_arm_hand_tcp_joint
- removed joint right_arm_joint1
- removed joint right_arm_joint2
- removed joint right_arm_joint3
- removed joint right_arm_joint4
- removed joint right_arm_joint5
- removed joint right_arm_joint6
- removed joint right_arm_joint7
- removed joint right_arm_joint8
- removed joint right_arm_joint_base
- removed joint right_arm_link0_sc_joint
- removed joint right_arm_link1_sc_joint
- removed joint right_arm_link2_sc_joint
- removed joint right_arm_link3_sc_joint
- removed joint right_arm_link4_sc_joint
- removed joint right_arm_link5_sc_joint
- removed joint right_arm_link6_sc_joint
- removed joint right_arm_link7_sc_joint
- added joint front_left_arm_finger_joint1: type prismatic, parent front_left_arm_hand, child front_left_arm_leftfinger, origin xyz=0 0 0.0584 rpy=0 0 0, axis 0 1 0, limit lower=0.0 upper=0.04 effort=100 velocity=0.2
- added joint front_left_arm_finger_joint2: type prismatic, parent front_left_arm_hand, child front_left_arm_rightfinger, origin xyz=0 0 0.0584 rpy=0 0 0, axis 0 -1 0, limit lower=0.0 upper=0.04 effort=100 velocity=0.2, mimic joint=front_left_arm_finger_joint1
- added joint front_left_arm_hand_joint: type fixed, parent front_left_arm_link8, child front_left_arm_hand, origin xyz=0 0 0 rpy=0 0 -0.7853981633974483
- added joint front_left_arm_hand_sc_joint: type fixed, parent front_left_arm_hand, child front_left_arm_hand_sc, origin rpy=0 0 0
- added joint front_left_arm_hand_tcp_joint: type fixed, parent front_left_arm_hand, child front_left_arm_hand_tcp, origin xyz=0 0 0.1034 rpy=0 0 0
- added joint front_left_arm_joint1: type revolute, parent front_left_arm_link0, child front_left_arm_link1, origin xyz=0 0 0.333 rpy=0 0 0, axis 0 0 1, limit lower=-2.8973 upper=2.8973 effort=87.0 velocity=2.175
- added joint front_left_arm_joint2: type revolute, parent front_left_arm_link1, child front_left_arm_link2, origin xyz=0 0 0 rpy=-1.5707963267948966 0 0, axis 0 0 1, limit lower=-1.7628 upper=1.7628 effort=87.0 velocity=2.175
- added joint front_left_arm_joint3: type revolute, parent front_left_arm_link2, child front_left_arm_link3, origin xyz=0 -0.316 0 rpy=1.5707963267948966 0 0, axis 0 0 1, limit lower=-2.8973 upper=2.8973 effort=87.0 velocity=2.175
- added joint front_left_arm_joint4: type revolute, parent front_left_arm_link3, child front_left_arm_link4, origin xyz=0.0825 0 0 rpy=1.5707963267948966 0 0, axis 0 0 1, limit lower=-3.0718 upper=-0.0698 effort=87.0 velocity=2.175
- added joint front_left_arm_joint5: type revolute, parent front_left_arm_link4, child front_left_arm_link5, origin xyz=-0.0825 0.384 0 rpy=-1.5707963267948966 0 0, axis 0 0 1, limit lower=-2.8973 upper=2.8973 effort=12.0 velocity=2.61
- added joint front_left_arm_joint6: type revolute, parent front_left_arm_link5, child front_left_arm_link6, origin xyz=0 0 0 rpy=1.5707963267948966 0 0, axis 0 0 1, limit lower=-0.0175 upper=3.7525 effort=12.0 velocity=2.61
- added joint front_left_arm_joint7: type revolute, parent front_left_arm_link6, child front_left_arm_link7, origin xyz=0.088 0 0 rpy=1.5707963267948966 0 0, axis 0 0 1, limit lower=-2.8973 upper=2.8973 effort=12.0 velocity=2.61
- added joint front_left_arm_joint8: type fixed, parent front_left_arm_link7, child front_left_arm_link8, origin xyz=0 0 0.107 rpy=0 0 0
- added joint front_left_arm_joint_base: type fixed, parent base, child front_left_arm_link0, origin xyz=0.5 0.5 1 rpy=0 0 0
- added joint front_left_arm_link0_sc_joint: type fixed, parent front_left_arm_link0, child front_left_arm_link0_sc, origin rpy=0 0 0
- added joint front_left_arm_link1_sc_joint: type fixed, parent front_left_arm_link1, child front_left_arm_link1_sc, origin rpy=0 0 0
- added joint front_left_arm_link2_sc_joint: type fixed, parent front_left_arm_link2, child front_left_arm_link2_sc, origin rpy=0 0 0
- added joint front_left_arm_link3_sc_joint: type fixed, parent front_left_arm_link3, child front_left_arm_link3_sc, origin rpy=0 0 0
- added joint front_left_arm_link4_sc_joint: type fixed, parent front_left_arm_link4, child front_left_arm_link4_sc, origin rpy=0 0 0
- added joint front_left_arm_link5_sc_joint: type fixed, parent front_left_arm_link5, child front_left_arm_link5_sc, origin rpy=0 0 0
- added joint front_left_arm_link6_sc_joint: type fixed, parent front_left_arm_link6, child front_left_arm_link6_sc, origin rpy=0 0 0
- added joint front_left_arm_link7_sc_joint: type fixed, parent front_left_arm_link7, child front_left_arm_link7_sc, origin rpy=0 0 0.7853981633974483
- added joint front_right_arm_finger_joint1: type prismatic, parent front_right_arm_hand, child front_right_arm_leftfinger, origin xyz=0 0 0.0584 rpy=0 0 0, axis 0 1 0, limit lower=0.0 upper=0.04 effort=100 velocity=0.2
- added joint front_right_arm_finger_joint2: type prismatic, parent front_right_arm_hand, child front_right_arm_rightfinger, origin xyz=0 0 0.0584 rpy=0 0 0, axis 0 -1 0, limit lower=0.0 upper=0.04 effort=100 velocity=0.2, mimic joint=front_right_arm_finger_joint1
- added joint front_right_arm_hand_joint: type fixed, parent front_right_arm_link8, child front_right_arm_hand, origin xyz=0 0 0 rpy=0 0 -0.7853981633974483
- added joint front_right_arm_hand_sc_joint: type fixed, parent front_right_arm_hand, child front_right_arm_hand_sc, origin rpy=0 0 0
- added joint front_right_arm_hand_tcp_joint: type fixed, parent front_right_arm_hand, child front_right_arm_hand_tcp, origin xyz=0 0 0.1034 rpy=0 0 0
- added joint front_right_arm_joint1: type revolute, parent front_right_arm_link0, child front_right_arm_link1, origin xyz=0 0 0.333 rpy=0 0 0, axis 0 0 1, limit lower=-2.8973 upper=2.8973 effort=87.0 velocity=2.175
- added joint front_right_arm_joint2: type revolute, parent front_right_arm_link1, child front_right_arm_link2, origin xyz=0 0 0 rpy=-1.5707963267948966 0 0, axis 0 0 1, limit lower=-1.7628 upper=1.7628 effort=87.0 velocity=2.175
- added joint front_right_arm_joint3: type revolute, parent front_right_arm_link2, child front_right_arm_link3, origin xyz=0 -0.316 0 rpy=1.5707963267948966 0 0, axis 0 0 1, limit lower=-2.8973 upper=2.8973 effort=87.0 velocity=2.175
- added joint front_right_arm_joint4: type revolute, parent front_right_arm_link3, child front_right_arm_link4, origin xyz=0.0825 0 0 rpy=1.5707963267948966 0 0, axis 0 0 1, limit lower=-3.0718 upper=-0.0698 effort=87.0 velocity=2.175
- added joint front_right_arm_joint5: type revolute, parent front_right_arm_link4, child front_right_arm_link5, origin xyz=-0.0825 0.384 0 rpy=-1.5707963267948966 0 0, axis 0 0 1, limit lower=-2.8973 upper=2.8973 effort=12.0 velocity=2.61
- added joint front_right_arm_joint6: type revolute, parent front_right_arm_link5, child front_right_arm_link6, origin xyz=0 0 0 rpy=1.5707963267948966 0 0, axis 0 0 1, limit lower=-0.0175 upper=3.7525 effort=12.0 velocity=2.61
- added joint front_right_arm_joint7: type revolute, parent front_right_arm_link6, child front_right_arm_link7, origin xyz=0.088 0 0 rpy=1.5707963267948966 0 0, axis 0 0 1, limit lower=-2.8973 upper=2.8973 effort=12.0 velocity=2.61
- added joint front_right_arm_joint8: type fixed, parent front_right_arm_link7, child front_right_arm_link8, origin xyz=0 0 0.107 rpy=0 0 0
- added joint front_right_arm_joint_base: type fixed, parent base, child front_right_arm_link0, origin xyz=0.5 -0.5 1 rpy=0 0 0
- added joint front_right_arm_link0_sc_joint: type fixed, parent front_right_arm_link0, child front_right_arm_link0_sc, origin rpy=0 0 0
- added joint front_right_arm_link1_sc_joint: type fixed, parent front_right_arm_link1, child front_right_arm_link1_sc, origin rpy=0 0 0
- added joint front_right_arm_link2_sc_joint: type fixed, parent front_right_arm_link2, child front_right_arm_link2_sc, origin rpy=0 0 0
- added joint front_right_arm_link3_sc_joint: type fixed, parent front_right_arm_link3, child front_right_arm_link3_sc, origin rpy=0 0 0
- added joint front_right_arm_link4_sc_joint: type fixed, parent front_right_arm_link4, child front_right_arm_link4_sc, origin rpy=0 0 0
- added joint front_right_arm_link5_sc_joint: type fixed, parent front_right_arm_link5, child front_right_arm_link5_sc, origin rpy=0 0 0
- added joint front_right_arm_link6_sc_joint: type fixed, parent front_right_arm_link6, child front_right_arm_link6_sc, origin rpy=0 0 0
- added joint front_right_arm_link7_sc_joint: type fixed, parent front_right_arm_link7, child front_right_arm_link7_sc, origin rpy=0 0 0.7853981633974483
- added joint rear_left_arm_finger_joint1: type prismatic, parent rear_left_arm_hand, child rear_left_arm_leftfinger, origin xyz=0 0 0.0584 rpy=0 0 0, axis 0 1 0, limit lower=0.0 upper=0.04 effort=100 velocity=0.2
- added joint rear_left_arm_finger_joint2: type prismatic, parent rear_left_arm_hand, child rear_left_arm_rightfinger, origin xyz=0 0 0.0584 rpy=0 0 0, axis 0 -1 0, limit lower=0.0 upper=0.04 effort=100 velocity=0.2, mimic joint=rear_left_arm_finger_joint1
- added joint rear_left_arm_hand_joint: type fixed, parent rear_left_arm_link8, child rear_left_arm_hand, origin xyz=0 0 0 rpy=0 0 -0.7853981633974483
- added joint rear_left_arm_hand_sc_joint: type fixed, parent rear_left_arm_hand, child rear_left_arm_hand_sc, origin rpy=0 0 0
- added joint rear_left_arm_hand_tcp_joint: type fixed, parent rear_left_arm_hand, child rear_left_arm_hand_tcp, origin xyz=0 0 0.1034 rpy=0 0 0
- added joint rear_left_arm_joint1: type revolute, parent rear_left_arm_link0, child rear_left_arm_link1, origin xyz=0 0 0.333 rpy=0 0 0, axis 0 0 1, limit lower=-2.8973 upper=2.8973 effort=87.0 velocity=2.175
- added joint rear_left_arm_joint2: type revolute, parent rear_left_arm_link1, child rear_left_arm_link2, origin xyz=0 0 0 rpy=-1.5707963267948966 0 0, axis 0 0 1, limit lower=-1.7628 upper=1.7628 effort=87.0 velocity=2.175
- added joint rear_left_arm_joint3: type revolute, parent rear_left_arm_link2, child rear_left_arm_link3, origin xyz=0 -0.316 0 rpy=1.5707963267948966 0 0, axis 0 0 1, limit lower=-2.8973 upper=2.8973 effort=87.0 velocity=2.175
- added joint rear_left_arm_joint4: type revolute, parent rear_left_arm_link3, child rear_left_arm_link4, origin xyz=0.0825 0 0 rpy=1.5707963267948966 0 0, axis 0 0 1, limit lower=-3.0718 upper=-0.0698 effort=87.0 velocity=2.175
- added joint rear_left_arm_joint5: type revolute, parent rear_left_arm_link4, child rear_left_arm_link5, origin xyz=-0.0825 0.384 0 rpy=-1.5707963267948966 0 0, axis 0 0 1, limit lower=-2.8973 upper=2.8973 effort=12.0 velocity=2.61
- added joint rear_left_arm_joint6: type revolute, parent rear_left_arm_link5, child rear_left_arm_link6, origin xyz=0 0 0 rpy=1.5707963267948966 0 0, axis 0 0 1, limit lower=-0.0175 upper=3.7525 effort=12.0 velocity=2.61
- added joint rear_left_arm_joint7: type revolute, parent rear_left_arm_link6, child rear_left_arm_link7, origin xyz=0.088 0 0 rpy=1.5707963267948966 0 0, axis 0 0 1, limit lower=-2.8973 upper=2.8973 effort=12.0 velocity=2.61
- added joint rear_left_arm_joint8: type fixed, parent rear_left_arm_link7, child rear_left_arm_link8, origin xyz=0 0 0.107 rpy=0 0 0
- added joint rear_left_arm_joint_base: type fixed, parent base, child rear_left_arm_link0, origin xyz=-0.5 0.5 1 rpy=0 0 0
- added joint rear_left_arm_link0_sc_joint: type fixed, parent rear_left_arm_link0, child rear_left_arm_link0_sc, origin rpy=0 0 0
- added joint rear_left_arm_link1_sc_joint: type fixed, parent rear_left_arm_link1, child rear_left_arm_link1_sc, origin rpy=0 0 0
- added joint rear_left_arm_link2_sc_joint: type fixed, parent rear_left_arm_link2, child rear_left_arm_link2_sc, origin rpy=0 0 0
- added joint rear_left_arm_link3_sc_joint: type fixed, parent rear_left_arm_link3, child rear_left_arm_link3_sc, origin rpy=0 0 0
- added joint rear_left_arm_link4_sc_joint: type fixed, parent rear_left_arm_link4, child rear_left_arm_link4_sc, origin rpy=0 0 0
- added joint rear_left_arm_link5_sc_joint: type fixed, parent rear_left_arm_link5, child rear_left_arm_link5_sc, origin rpy=0 0 0
- added joint rear_left_arm_link6_sc_joint: type fixed, parent rear_left_arm_link6, child rear_left_arm_link6_sc, origin rpy=0 0 0
- added joint rear_left_arm_link7_sc_joint: type fixed, parent rear_left_arm_link7, child rear_left_arm_link7_sc, origin rpy=0 0 0.7853981633974483
- added joint rear_right_arm_finger_joint1: type prismatic, parent rear_right_arm_hand, child rear_right_arm_leftfinger, origin xyz=0 0 0.0584 rpy=0 0 0, axis 0 1 0, limit lower=0.0 upper=0.04 effort=100 velocity=0.2
- added joint rear_right_arm_finger_joint2: type prismatic, parent rear_right_arm_hand, child rear_right_arm_rightfinger, origin xyz=0 0 0.0584 rpy=0 0 0, axis 0 -1 0, limit lower=0.0 upper=0.04 effort=100 velocity=0.2, mimic joint=rear_right_arm_finger_joint1
- added joint rear_right_arm_hand_joint: type fixed, parent rear_right_arm_link8, child rear_right_arm_hand, origin xyz=0 0 0 rpy=0 0 -0.7853981633974483
- added joint rear_right_arm_hand_sc_joint: type fixed, parent rear_right_arm_hand, child rear_right_arm_hand_sc, origin rpy=0 0 0
- added joint rear_right_arm_hand_tcp_joint: type fixed, parent rear_right_arm_hand, child rear_right_arm_hand_tcp, origin xyz=0 0 0.1034 rpy=0 0 0
- added joint rear_right_arm_joint1: type revolute, parent rear_right_arm_link0, child rear_right_arm_link1, origin xyz=0 0 0.333 rpy=0 0 0, axis 0 0 1, limit lower=-2.8973 upper=2.8973 effort=87.0 velocity=2.175
- added joint rear_right_arm_joint2: type revolute, parent rear_right_arm_link1, child rear_right_arm_link2, origin xyz=0 0 0 rpy=-1.5707963267948966 0 0, axis 0 0 1, limit lower=-1.7628 upper=1.7628 effort=87.0 velocity=2.175
- added joint rear_right_arm_joint3: type revolute, parent rear_right_arm_link2, child rear_right_arm_link3, origin xyz=0 -0.316 0 rpy=1.5707963267948966 0 0, axis 0 0 1, limit lower=-2.8973 upper=2.8973 effort=87.0 velocity=2.175
- added joint rear_right_arm_joint4: type revolute, parent rear_right_arm_link3, child rear_right_arm_link4, origin xyz=0.0825 0 0 rpy=1.5707963267948966 0 0, axis 0 0 1, limit lower=-3.0718 upper=-0.0698 effort=87.0 velocity=2.175
- added joint rear_right_arm_joint5: type revolute, parent rear_right_arm_link4, child rear_right_arm_link5, origin xyz=-0.0825 0.384 0 rpy=-1.5707963267948966 0 0, axis 0 0 1, limit lower=-2.8973 upper=2.8973 effort=12.0 velocity=2.61
- added joint rear_right_arm_joint6: type revolute, parent rear_right_arm_link5, child rear_right_arm_link6, origin xyz=0 0 0 rpy=1.5707963267948966 0 0, axis 0 0 1, limit lower=-0.0175 upper=3.7525 effort=12.0 velocity=2.61
- added joint rear_right_arm_joint7: type revolute, parent rear_right_arm_link6, child rear_right_arm_link7, origin xyz=0.088 0 0 rpy=1.5707963267948966 0 0, axis 0 0 1, limit lower=-2.8973 upper=2.8973 effort=12.0 velocity=2.61
- added joint rear_right_arm_joint8: type fixed, parent rear_right_arm_link7, child rear_right_arm_link8, origin xyz=0 0 0.107 rpy=0 0 0
- added joint rear_right_arm_joint_base: type fixed, parent base, child rear_right_arm_link0, origin xyz=-0.5 -0.5 1 rpy=0 0 0
- added joint rear_right_arm_link0_sc_joint: type fixed, parent rear_right_arm_link0, child rear_right_arm_link0_sc, origin rpy=0 0 0
- added joint rear_right_arm_link1_sc_joint: type fixed, parent rear_right_arm_link1, child rear_right_arm_link1_sc, origin rpy=0 0 0
- added joint rear_right_arm_link2_sc_joint: type fixed, parent rear_right_arm_link2, child rear_right_arm_link2_sc, origin rpy=0 0 0
- added joint rear_right_arm_link3_sc_joint: type fixed, parent rear_right_arm_link3, child rear_right_arm_link3_sc, origin rpy=0 0 0
- added joint rear_right_arm_link4_sc_joint: type fixed, parent rear_right_arm_link4, child rear_right_arm_link4_sc, origin rpy=0 0 0
- added joint rear_right_arm_link5_sc_joint: type fixed, parent rear_right_arm_link5, child rear_right_arm_link5_sc, origin rpy=0 0 0
- added joint rear_right_arm_link6_sc_joint: type fixed, parent rear_right_arm_link6, child rear_right_arm_link6_sc, origin rpy=0 0 0
- added joint rear_right_arm_link7_sc_joint: type fixed, parent rear_right_arm_link7, child rear_right_arm_link7_sc, origin rpy=0 0 0.7853981633974483
