Commit message: Added 4 robots simulation and initial documentation

File: ke_ws/src/panda_multiple_arms/robot_description/panda_multiple_arms.xacro (robot description, xacro)
@@ -2,6 +2,8 @@
 <robot name="panda_multiple_arms" xmlns:xacro="http://ros.org/wiki/xacro">
     <!-- add arms names prefixes -->
-    <xacro:arg name="arm_id_1" default="right_arm" />
-    <xacro:arg name="arm_id_2" default="left_arm" />
+    <xacro:arg name="arm_id_1" default="front_right_arm" />
+    <xacro:arg name="arm_id_2" default="front_left_arm" />
+    <xacro:arg name="arm_id_3" default="rear_right_arm" />
+    <xacro:arg name="arm_id_4" default="rear_left_arm" />
     <!-- load arm/hand models and utils (which adds the robot inertia tags to be Gazebo-simulation ready) -->
     <xacro:include filename="$(find franka_description)/robots/common/utils.xacro" />
@@ -14,5 +16,5 @@
             <origin xyz="0 0 0.5" rpy="0 0 0" />
             <geometry>
-                <box size="1 2 1" />
+                <box size="2 2 1" />
             </geometry>
             <material name="White">
@@ -23,10 +25,10 @@
             <origin xyz="0 0 0.5" rpy="0 0 0" />
             <geometry>
-                <box size="1 2 1" />
+                <box size="2 2 1" />
             </geometry>
         </collision>
         <inertial>
             <origin xyz="0.0 0.0 0.0" rpy="0.0 0.0 0.0"/>
-            <mass value="10.0"/>
+            <mass value="20.0"/>
             <inertia ixx="0.001" ixy="0.0" ixz="0.001" iyy="0.0" iyz="0.0" izz="0.001"/>
         </inertial>
@@ -37,11 +39,17 @@
         <origin xyz="0.0 0.0 0.0" rpy="0.0 0.0 0.0"/>
     </joint>
-    <!-- right arm with gripper -->
-    <xacro:franka_arm arm_id="$(arg arm_id_1)" connected_to="base" xyz="0 -0.5 1" gazebo="true" safety_distance="0.03" joint_limits="${xacro.load_yaml('$(find franka_description)/robots/panda/joint_limits.yaml')}"/>
+    <!-- front right arm with gripper -->
+    <xacro:franka_arm arm_id="$(arg arm_id_1)" connected_to="base" xyz="0.5 -0.5 1" gazebo="true" safety_distance="0.03" joint_limits="${xacro.load_yaml('$(find franka_description)/robots/panda/joint_limits.yaml')}"/>
     <xacro:franka_hand arm_id="$(arg arm_id_1)" rpy="0 0 ${-pi/4}" connected_to="$(arg arm_id_1)_link8" gazebo="true" safety_distance="0.03" />
-    <!-- left arm with gripper -->
-    <xacro:franka_arm arm_id="$(arg arm_id_2)" connected_to="base" xyz="0 0.5 1" gazebo="true" safety_distance="0.03" joint_limits="${xacro.load_yaml('$(find franka_description)/robots/panda/joint_limits.yaml')}"/>
+    <!-- front left arm with gripper -->
+    <xacro:franka_arm arm_id="$(arg arm_id_2)" connected_to="base" xyz="0.5 0.5 1" gazebo="true" safety_distance="0.03" joint_limits="${xacro.load_yaml('$(find franka_description)/robots/panda/joint_limits.yaml')}"/>
     <xacro:franka_hand arm_id="$(arg arm_id_2)" rpy="0 0 ${-pi/4}" connected_to="$(arg arm_id_2)_link8" gazebo="true" safety_distance="0.03" />
-    <!-- right arm joints control interface -->
+    <!-- rear right arm with gripper -->
+    <xacro:franka_arm arm_id="$(arg arm_id_3)" connected_to="base" xyz="-0.5 -0.5 1" gazebo="true" safety_distance="0.03" joint_limits="${xacro.load_yaml('$(find franka_description)/robots/panda/joint_limits.yaml')}"/>
+    <xacro:franka_hand arm_id="$(arg arm_id_3)" rpy="0 0 ${-pi/4}" connected_to="$(arg arm_id_3)_link8" gazebo="true" safety_distance="0.03" />
+    <!-- rear left arm with gripper -->
+    <xacro:franka_arm arm_id="$(arg arm_id_4)" connected_to="base" xyz="-0.5 0.5 1" gazebo="true" safety_distance="0.03" joint_limits="${xacro.load_yaml('$(find franka_description)/robots/panda/joint_limits.yaml')}"/>
+    <xacro:franka_hand arm_id="$(arg arm_id_4)" rpy="0 0 ${-pi/4}" connected_to="$(arg arm_id_4)_link8" gazebo="true" safety_distance="0.03" />
+    <!-- front right arm joints control interface -->
     <xacro:gazebo-joint joint="$(arg arm_id_1)_joint1" transmission="hardware_interface/PositionJointInterface" />
     <xacro:gazebo-joint joint="$(arg arm_id_1)_joint2" transmission="hardware_interface/PositionJointInterface" />
@@ -51,5 +59,5 @@
     <xacro:gazebo-joint joint="$(arg arm_id_1)_joint6" transmission="hardware_interface/PositionJointInterface" />
     <xacro:gazebo-joint joint="$(arg arm_id_1)_joint7" transmission="hardware_interface/PositionJointInterface" />
-    <!-- left arm joints control interface -->
+    <!-- front left arm joints control interface -->
     <xacro:gazebo-joint joint="$(arg arm_id_2)_joint1" transmission="hardware_interface/PositionJointInterface" />
     <xacro:gazebo-joint joint="$(arg arm_id_2)_joint2" transmission="hardware_interface/PositionJointInterface" />
@@ -59,4 +67,20 @@
     <xacro:gazebo-joint joint="$(arg arm_id_2)_joint6" transmission="hardware_interface/PositionJointInterface" />
     <xacro:gazebo-joint joint="$(arg arm_id_2)_joint7" transmission="hardware_interface/PositionJointInterface" />
+    <!-- rear right arm joints control interface -->
+    <xacro:gazebo-joint joint="$(arg arm_id_3)_joint1" transmission="hardware_interface/PositionJointInterface" />
+    <xacro:gazebo-joint joint="$(arg arm_id_3)_joint2" transmission="hardware_interface/PositionJointInterface" />
+    <xacro:gazebo-joint joint="$(arg arm_id_3)_joint3" transmission="hardware_interface/PositionJointInterface" />
+    <xacro:gazebo-joint joint="$(arg arm_id_3)_joint4" transmission="hardware_interface/PositionJointInterface" />
+    <xacro:gazebo-joint joint="$(arg arm_id_3)_joint5" transmission="hardware_interface/PositionJointInterface" />
+    <xacro:gazebo-joint joint="$(arg arm_id_3)_joint6" transmission="hardware_interface/PositionJointInterface" />
+    <xacro:gazebo-joint joint="$(arg arm_id_3)_joint7" transmission="hardware_interface/PositionJointInterface" />
+    <!-- rear left arm joints control interface -->
+    <xacro:gazebo-joint joint="$(arg arm_id_4)_joint1" transmission="hardware_interface/PositionJointInterface" />
+    <xacro:gazebo-joint joint="$(arg arm_id_4)_joint2" transmission="hardware_interface/PositionJointInterface" />
+    <xacro:gazebo-joint joint="$(arg arm_id_4)_joint3" transmission="hardware_interface/PositionJointInterface" />
+    <xacro:gazebo-joint joint="$(arg arm_id_4)_joint4" transmission="hardware_interface/PositionJointInterface" />
+    <xacro:gazebo-joint joint="$(arg arm_id_4)_joint5" transmission="hardware_interface/PositionJointInterface" />
+    <xacro:gazebo-joint joint="$(arg arm_id_4)_joint6" transmission="hardware_interface/PositionJointInterface" />
+    <xacro:gazebo-joint joint="$(arg arm_id_4)_joint7" transmission="hardware_interface/PositionJointInterface" />
     <!-- right hand joints control interface -->
     <xacro:gazebo-joint joint="$(arg arm_id_1)_finger_joint1" transmission="hardware_interface/EffortJointInterface" />
@@ -65,4 +89,10 @@
     <xacro:gazebo-joint joint="$(arg arm_id_2)_finger_joint1" transmission="hardware_interface/EffortJointInterface" />
     <xacro:gazebo-joint joint="$(arg arm_id_2)_finger_joint2" transmission="hardware_interface/EffortJointInterface" />
+    <!-- right hand joints control interface -->
+    <xacro:gazebo-joint joint="$(arg arm_id_3)_finger_joint1" transmission="hardware_interface/EffortJointInterface" />
+    <xacro:gazebo-joint joint="$(arg arm_id_3)_finger_joint2" transmission="hardware_interface/EffortJointInterface" />
+    <!-- left hand joints control interface -->
+    <xacro:gazebo-joint joint="$(arg arm_id_4)_finger_joint1" transmission="hardware_interface/EffortJointInterface" />
+    <xacro:gazebo-joint joint="$(arg arm_id_4)_finger_joint2" transmission="hardware_interface/EffortJointInterface" />
     <!-- load ros_control plugin -->
     <gazebo>
